Commit message: 将guguji_ros2原始内容移植到ros2系统下可以正常启动的软件包，其中在rviz和gazebo中都可以正常打开

File: guguji_ros2_ws/src/guguji_ros2/urdf/guguji.urdf (robot description, URDF)
Before this commit: robot guguji, 9 links, 8 joints
Links:
- link base_link: geometry collision mesh filename=package://guguji_ros2/meshes/base_link.STL; visual mesh filename=package://guguji_ros2/meshes/base_link.STL
- link left_ankle_pitch_link: geometry collision mesh filename=package://guguji_ros2/meshes/left_ankle_pitch_link.STL; visual mesh filename=package://guguji_ros2/meshes/left_ankle_pitch_link.STL
- link left_foot_link: geometry collision mesh filename=package://guguji_ros2/meshes/left_foot_link.STL; visual mesh filename=package://guguji_ros2/meshes/left_foot_link.STL
- link left_hip_pitch_link: geometry collision mesh filename=package://guguji_ros2/meshes/left_hip_pitch_link.STL; visual mesh filename=package://guguji_ros2/meshes/left_hip_pitch_link.STL
- link left_knee_pitch_link: geometry collision mesh filename=package://guguji_ros2/meshes/left_knee_pitch_link.STL; visual mesh filename=package://guguji_ros2/meshes/left_knee_pitch_link.STL
- link right_ankle_pitch_link: geometry collision mesh filename=package://guguji_ros2/meshes/right_ankle_pitch_link.STL; visual mesh filename=package://guguji_ros2/meshes/right_ankle_pitch_link.STL
- link right_foot_link: geometry collision mesh filename=package://guguji_ros2/meshes/right_foot_link.STL; visual mesh filename=package://guguji_ros2/meshes/right_foot_link.STL
- link right_hip_pitch_link: geometry collision mesh filename=package://guguji_ros2/meshes/right_hip_pitch_link.STL; visual mesh filename=package://guguji_ros2/meshes/right_hip_pitch_link.STL
- link right_knee_pitch_link: geometry collision mesh filename=package://guguji_ros2/meshes/right_knee_pitch_link.STL; visual mesh filename=package://guguji_ros2/meshes/right_knee_pitch_link.STL
Joints:
- removed joint eft_hip_pitch_joint
- added joint left_hip_pitch_joint: type revolute, parent base_link, child left_hip_pitch_link, origin xyz=0.0212 0.075 -0.045 rpy=0 0 0, axis -1 0 -8.3367E-05, limit lower=0 upper=0 effort=0 velocity=0
- joint right_ankle_pitch_joint: limit (none) -> lower=0 upper=0 effort=0 velocity=0; type continuous -> revolute

Commit message: 更新guguji.urdf文件，使其可以在rivz中正常进行关节控制

File: guguji_ros2_ws/src/guguji_ros2/urdf/guguji.urdf (robot description, URDF)
Before this commit: robot guguji, 9 links, 8 joints
Joints:
- joint left_ankle_joint: limit lower=0 upper=0 effort=0 velocity=0 -> lower=-0.6 upper=0.6 effort=8.0 velocity=2.0
- joint left_ankle_pitch_joint: limit lower=0 upper=0 effort=0 velocity=0 -> lower=-0.8 upper=0.8 effort=8.0 velocity=2.0
- joint left_hip_pitch_joint: limit lower=0 upper=0 effort=0 velocity=0 -> lower=-1.0 upper=1.0 effort=10.0 velocity=2.0
- joint left_knee_pitch_joint: limit lower=0 upper=0 effort=0 velocity=0 -> lower=-1.2 upper=1.2 effort=10.0 velocity=2.0
- joint right_ankle_joint: limit lower=0 upper=0 effort=0 velocity=0 -> lower=-0.6 upper=0.6 effort=8.0 velocity=2.0
- joint right_ankle_pitch_joint: limit lower=0 upper=0 effort=0 velocity=0 -> lower=-0.8 upper=0.8 effort=8.0 velocity=2.0
- joint right_hip_pitch_joint: limit lower=0 upper=0 effort=0 velocity=0 -> lower=-1.0 upper=1.0 effort=10.0 velocity=2.0
- joint right_knee_pitch_joint: limit lower=0 upper=0 effort=0 velocity=0 -> lower=-1.2 upper=1.2 effort=10.0 velocity=2.0
